File: src/PCB/mainpcb.kicad_pcb (KiCad board)
At the start: 2 copper layers, 69.8 x 45.7 mm, 9 parts, among them CON1 BARREL_JACK, P1 VALVE1, P2 VALVE2, Q1 PN2222A, Q2 PN2222A, U1 LM317T, U2 Adafruit_HUZZAH

Commit message: pcb
Parts:
- removed R1: 370, Resistors_ThroughHole:Resistor_Horizontal_RM7mm
- added R11: 330, Resistors_ThroughHole:Resistor_Horizontal_RM7mm, F.Cu at (63.5, 24.1)
- added R12: 39, Resistors_ThroughHole:Resistor_Horizontal_RM7mm, F.Cu at (63.5, 35.6)
Connections:
- CON1 pad 3: Net-(CON1-Pad2) -> Net-(CON1-Pad3)
Routing:
- net Net-(R11-Pad2): track 0.00 -> 3.81 mm
- net Net-(R12-Pad2): track 8.89 -> 10.5 mm
- net Net-(P1-Pad1): track 56.2 -> 56.9 mm

Commit message: power and ground plane
Connections:
- net Net-(CON1-Pad2) renamed GND
- net Net-(P1-Pad1) renamed +12V
Routing:
- added copper zone on F.Cu, net +12V
- added copper zone on B.Cu, net GND
