File: src/PCB/mainpcb.sch (KiCad schematic (older format))
At the start: 9 parts, among them CON1 BARREL_JACK, P1 VALVE1, P2 VALVE2, Q1 PN2222A, Q2 PN2222A, U1 LM317T, U2 Adafruit_HUZZAH

Commit message: pcb
Parts:
- added R12: 39, Resistors_ThroughHole:Resistor_Horizontal_RM7mm, symbol R
- R11: renamed from R1; value 370 -> 330
Connections:
- net at CON1.2, Q1.1 (E), Q2.1 (E)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: no longer CON1.3
- net at R2.1, U1.1 (ADJ): now also R12.2; no longer R11.2
- new net: R11.2, R12.1
Other:
- moved on the sheet: R2, U2
Changed lines of the file:
@@
 $EndComp
 $Comp
-L R R1
+L R R11
 U 1 1 56F82978
 P 4000 1950
-F 0 "R1" V 4080 1950 50  0000 C CNN
-F 1 "370" V 4000 1950 50  0000 C CNN
+F 0 "R11" V 4080 1950 50  0000 C CNN
+F 1 "330" V 4000 1950 50  0000 C CNN
 F 2 "Resistors_ThroughHole:Resistor_Horizontal_RM7mm" V 3930 1950 50  0001 C CNN
 F 3 "" H 4000 1950 50  0000 C CNN
@@
 L R R2
 U 1 1 56F829DB
-P 4000 2400
-F 0 "R2" V 4080 2400 50  0000 C CNN
-F 1 "3300" V 4000 2400 50  0000 C CNN
-F 2 "Resistors_ThroughHole:Resistor_Horizontal_RM7mm" V 3930 2400 50  0001 C CNN
-F 3 "" H 4000 2400 50  0000 C CNN
-	1    4000 2400
+P 4000 2650
+F 0 "R2" V 4080 2650 50  0000 C CNN
+F 1 "3300" V 4000 2650 50  0000 C CNN
+F 2 "Resistors_ThroughHole:Resistor_Horizontal_RM7mm" V 3930 2650 50  0001 C CNN
+F 3 "" H 4000 2650 50  0000 C CNN
+	1    4000 2650
 	1    0    0    -1
 $EndComp
@@
 L Adafruit_HUZZAH U2
 U 1 1 56F82B44
-P 5150 3300
-F 0 "U2" H 5150 2700 60  0000 C CNN
-F 1 "Adafruit_HUZZAH" H 5150 3900 60  0000 C CNN
-F 2 "Adafruit_huzzah:Adafruit HUZZAH" H 5050 2950 60  0001 C CNN
-F 3 "" H 5050 2950 60  0000 C CNN
-	1    5150 3300
+P 5500 3550
+F 0 "U2" H 5500 2950 60  0000 C CNN
+F 1 "Adafruit_HUZZAH" H 5500 4150 60  0000 C CNN
+F 2 "Adafruit_huzzah:Adafruit HUZZAH" H 5400 3200 60  0001 C CNN
+F 3 "" H 5400 3200 60  0000 C CNN
+	1    5500 3550
 	1    0    0    -1
 $EndComp
 Wire Wire Line
-	3950 1750 5100 1750
-Wire Wire Line
-	4000 1750 4000 1800
-Wire Wire Line
-	4000 2100 4000 2250
-Wire Wire Line
-	3550 2050 3550 2150
-Wire Wire Line
-	3550 2150 4000 2150
-Connection ~ 4000 2150
-Wire Wire Line
 	2750 1750 3150 1750
-Wire Wire Line
-	2750 2550 6100 2550
 $Comp
 L CONN_01X02 P1
@@
 	0    -1   -1   0
 $EndComp
-Connection ~ 4000 1750
 Wire Wire Line
 	5200 1750 5200 1900
 Wire Wire Line
-	6000 1750 6000 1800
-Wire Wire Line
-	6000 1800 4000 1800
-Wire Wire Line
 	6100 1750 6100 1900
 Wire Wire Line
-	5200 2550 5200 2300
-Connection ~ 4000 2550
+	5200 2800 5200 2300
 Wire Wire Line
-	6100 2550 6100 2300
-Connection ~ 5200 2550
-Connection ~ 2750 2550
+	6100 2800 6100 2300
+Connection ~ 2750 1950
+$Comp
+L R R12
+U 1 1 56F87A89
+P 4000 2300
+F 0 "R12" V 4080 2300 50  0000 C CNN
+F 1 "39" V 4000 2300 50  0000 C CNN
+F 2 "Resistors_ThroughHole:Resistor_Horizontal_RM7mm" V 3930 2300 50  0001 C CNN
+F 3 "" H 4000 2300 50  0000 C CNN
+	1    4000 2300
+	1    0    0    -1
+$EndComp
 Wire Wire Line
-	2750 1850 2750 3750
-Connection ~ 2750 1950
+	4000 2100 4000 2150
 Wire Wire Line
-	2750 3750 4550 3750
+	4000 2450 4000 2500
 Wire Wire Line
-	4550 3550 4200 3550
+	3550 2050 3550 2500
 Wire Wire Line
-	4200 3550 4200 1750
-Connection ~ 4200 1750
+	3550 2500 4000 2500
 Wire Wire Line
-	4900 2100 4250 2100
+	2750 1950 2750 2800
 Wire Wire Line
-	4250 2100 4250 3250
+	2750 2800 6100 2800
+Connection ~ 4000 2800
+Connection ~ 5200 2800
 Wire Wire Line
-	4250 3250 4550 3250
+	3950 1750 6000 1750
 Wire Wire Line
-	5800 2100 5800 2500
+	4000 1750 4000 1800
+Connection ~ 4000 1750
+Connection ~ 5100 1750
 Wire Wire Line
-	5800 2500 4300 2500
+	4900 3800 4300 3800
 Wire Wire Line
-	4300 2500 4300 3150
+	4300 3800 4300 1750
+Connection ~ 4300 1750
 Wire Wire Line
-	4300 3150 4550 3150
+	4900 4000 4350 4000
+Wire Wire Line
+	4350 4000 4350 2800
+Connection ~ 4350 2800
+Wire Wire Line
+	4900 2100 4600 2100
+Wire Wire Line
+	4600 2100 4600 3500
+Wire Wire Line
+	4600 3500 4900 3500
+Wire Wire Line
+	5800 2100 5800 2750
+Wire Wire Line
+	5800 2750 4650 2750
+Wire Wire Line
+	4650 2750 4650 3400
+Wire Wire Line
+	4650 3400 4900 3400
 $EndSCHEMATC

Commit message: power and ground plane
Connections:
- net GND: now reaches CON1.2, Q1.1 (E), Q2.1 (E), R2.2, U2.19 (GND)
- net +12V: now reaches P1.1 (P1), P2.1 (P1), R11.1, U1.2 (OUT), U2.15 (VIN)
Changed lines of the file:
@@
 LIBS:contrib
 LIBS:valves
-LIBS:adafruit_huzzah
 LIBS:mainpcb-cache
 EELAYER 25 0
@@
 	3550 2500 4000 2500
 Wire Wire Line
-	2750 1950 2750 2800
+	2750 1950 2750 3000
 Wire Wire Line
 	2750 2800 6100 2800
@@
 Connection ~ 5100 1750
 Wire Wire Line
-	4900 3800 4300 3800
-Wire Wire Line
-	4300 3800 4300 1750
+	4300 3800 4900 3800
+Wire Wire Line
+	4300 1450 4300 3800
 Connection ~ 4300 1750
 Wire Wire Line
@@
 Wire Wire Line
 	4650 3400 4900 3400
+$Comp
+L GND #PWR?
+U 1 1 56FAB0DF
+P 2750 3000
+F 0 "#PWR?" H 2750 2750 50  0001 C CNN
+F 1 "GND" H 2750 2850 50  0000 C CNN
+F 2 "" H 2750 3000 50  0000 C CNN
+F 3 "" H 2750 3000 50  0000 C CNN
+	1    2750 3000
+	1    0    0    -1
+$EndComp
+Connection ~ 2750 2800
+$Comp
+L +12V #PWR?
+U 1 1 56FAB133
+P 4300 1450
+F 0 "#PWR?" H 4300 1300 50  0001 C CNN
+F 1 "+12V" H 4300 1590 50  0000 C CNN
+F 2 "" H 4300 1450 50  0000 C CNN
+F 3 "" H 4300 1450 50  0000 C CNN
+	1    4300 1450
+	1    0    0    -1
+$EndComp
 $EndSCHEMATC
