File: PCB/mainpcb.kicad_pcb (KiCad board)
At the start: 2 copper layers, 69.8 x 45.7 mm, 10 parts, among them CON1 BARREL_JACK, P1 VALVE1, P2 VALVE2, Q1 PN2222A, Q2 PN2222A, U1 LM317T, U2 Adafruit_HUZZAH

Commit message: pcb changes
Parts:
- moved P1 41.4 mm to (50.8, 57.7), turned to 90 degrees
- moved P2 37.8 mm to (67.6, 57.7), turned to 90 degrees
Routing:
- net +12V: track 56.9 -> 111.1 mm
- net Net-(P1-Pad2): track 14.0 -> 35.0 mm
- net Net-(P2-Pad2): track 14.5 -> 25.7 mm
Changed lines of the file:
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@@
     (links 16)
     (no_connects 0)
-    (area 39.294999 16.434999 109.295001 62.305001)
+    (area 27.560001 14.46552 109.495001 70.010001)
     (thickness 1.6)
     (drawings 6)
-    (tracks 29)
+    (tracks 37)
     (zones 0)
     (modules 10)
@@
   )
   (module Pin_Headers:Pin_Header_Straight_1x02 (layer F.Cu)
-    (at 68.58 20.32)
+    (at 50.8 57.658 90)
     (descr "Through hole pin header")
     (tags "pin header")
-    (fp_text reference P1 (at -2.54 -1.27) (layer F.SilkS)
-      (effects (font (size 1 1) (thickness 0.15)))
-    )
-    (fp_text value VALVE1 (at 0 -2.54) (layer F.Fab)
+    (fp_text reference P1 (at -1.27 5.588 180) (layer F.SilkS)
+      (effects (font (size 1 1) (thickness 0.15)))
+    )
+    (fp_text value VALVE1 (at 2.794 1.524 180) (layer F.Fab)
       (effects (font (size 1 1) (thickness 0.15)))
     )
@@
     (fp_line (start -1.27 1.27) (end -1.27 3.81) (layer F.SilkS) (width 0.15))
     (fp_line (start -1.27 3.81) (end 1.27 3.81) (layer F.SilkS) (width 0.15))
-    (pad 1 thru_hole rect (at 0 0) (size 2.032 2.032) (drill 1.016) (layers *.Cu *.Mask F.SilkS)
+    (pad 1 thru_hole rect (at 0 0 90) (size 2.032 2.032) (drill 1.016) (layers *.Cu *.Mask F.SilkS)
       (net 26 +12V))
-    (pad 2 thru_hole oval (at 0 2.54) (size 2.032 2.032) (drill 1.016) (layers *.Cu *.Mask F.SilkS)
+    (pad 2 thru_hole oval (at 0 2.54 90) (size 2.032 2.032) (drill 1.016) (layers *.Cu *.Mask F.SilkS)
       (net 2 "Net-(P1-Pad2)"))
     (model Pin_Headers.3dshapes/Pin_Header_Straight_1x02.wrl
@@
   )
   (module Pin_Headers:Pin_Header_Straight_1x02 (layer F.Cu)
-    (at 73.66 20.32)
+    (at 67.564 57.658 90)
     (descr "Through hole pin header")
     (tags "pin header")
-    (fp_text reference P2 (at 3.81 -1.27) (layer F.SilkS)
-      (effects (font (size 1 1) (thickness 0.15)))
-    )
-    (fp_text value VALVE2 (at 1.27 -2.54) (layer F.Fab)
+    (fp_text reference P2 (at -1.27 5.588 180) (layer F.SilkS)
+      (effects (font (size 1 1) (thickness 0.15)))
+    )
+    (fp_text value VALVE2 (at 2.794 1.27 180) (layer F.Fab)
       (effects (font (size 1 1) (thickness 0.15)))
     )
@@
     (fp_line (start -1.27 1.27) (end -1.27 3.81) (layer F.SilkS) (width 0.15))
     (fp_line (start -1.27 3.81) (end 1.27 3.81) (layer F.SilkS) (width 0.15))
-    (pad 1 thru_hole rect (at 0 0) (size 2.032 2.032) (drill 1.016) (layers *.Cu *.Mask F.SilkS)
+    (pad 1 thru_hole rect (at 0 0 90) (size 2.032 2.032) (drill 1.016) (layers *.Cu *.Mask F.SilkS)
       (net 26 +12V))
-    (pad 2 thru_hole oval (at 0 2.54) (size 2.032 2.032) (drill 1.016) (layers *.Cu *.Mask F.SilkS)
+    (pad 2 thru_hole oval (at 0 2.54 90) (size 2.032 2.032) (drill 1.016) (layers *.Cu *.Mask F.SilkS)
       (net 3 "Net-(P2-Pad2)"))
     (model Pin_Headers.3dshapes/Pin_Header_Straight_1x02.wrl
@@
   (gr_line (start 39.37 16.51) (end 39.37 62.23) (angle 90) (layer Edge.Cuts) (width 0.15))
   (segment (start 53.19014 21.59) (end 59.69 21.59) (width 0.25) (layer F.Cu) (net 1))
-  (segment (start 68.58 22.86) (end 68.58 36.83) (width 0.25) (layer F.Cu) (net 2))
-  (segment (start 73.66 22.86) (end 73.66 35.56) (width 0.25) (layer F.Cu) (net 3))
-  (segment (start 73.66 35.56) (end 74.93 36.83) (width 0.25) (layer F.Cu) (net 3))
+  (segment (start 68.58 36.83) (end 65.024 36.83) (width 0.25) (layer B.Cu) (net 2) (status 400000))
+  (segment (start 63.246 57.658) (end 53.34 57.658) (width 0.25) (layer B.Cu) (net 2) (status 800000))
+  (segment (start 63.246 38.608) (end 63.246 57.658) (width 0.25) (layer B.Cu) (net 2))
+  (segment (start 65.024 36.83) (end 63.246 38.608) (width 0.25) (layer B.Cu) (net 2))
+  (segment (start 74.93 36.83) (end 73.152 36.83) (width 0.25) (layer B.Cu) (net 3) (status 400000))
+  (segment (start 73.152 57.658) (end 70.104 57.658) (width 0.25) (layer B.Cu) (net 3) (status 800000))
+  (segment (start 73.152 36.83) (end 73.152 57.658) (width 0.25) (layer B.Cu) (net 3))
   (segment (start 68.58 38.1) (end 71.12 38.1) (width 0.25) (layer B.Cu) (net 4))
   (segment (start 71.12 35.56) (end 86.36 35.56) (width 0.25) (layer B.Cu) (net 4))
@@
   (segment (start 52.07 31.75) (end 52.07 39.37) (width 0.25) (layer F.Cu) (net 25))
   (segment (start 52.07 39.37) (end 68.58 39.37) (width 0.25) (layer F.Cu) (net 25))
-  (segment (start 63.5 24.13) (end 63.5 22.86) (width 0.25) (layer F.Cu) (net 26))
-  (segment (start 66.04 20.32) (end 68.58 20.32) (width 0.25) (layer F.Cu) (net 26))
-  (segment (start 63.5 22.86) (end 66.04 20.32) (width 0.25) (layer F.Cu) (net 26))
+  (segment (start 86.36 43.18) (end 88.646 43.18) (width 0.25) (layer F.Cu) (net 26) (status 400000))
+  (segment (start 88.646 60.452) (end 67.564 60.452) (width 0.25) (layer F.Cu) (net 26))
+  (segment (start 88.646 43.18) (end 88.646 60.452) (width 0.25) (layer F.Cu) (net 26))
+  (segment (start 50.8 57.658) (end 50.8 60.452) (width 0.25) (layer F.Cu) (net 26) (status 400000))
+  (segment (start 67.564 60.452) (end 67.564 57.658) (width 0.25) (layer F.Cu) (net 26) (status 800000))
+  (segment (start 50.8 60.452) (end 67.564 60.452) (width 0.25) (layer F.Cu) (net 26))
+  (segment (start 59.69 24.13) (end 57.15 24.13) (width 0.25) (layer B.Cu) (net 26) (status 400000))
+  (segment (start 47.117 57.658) (end 50.8 57.658) (width 0.25) (layer B.Cu) (net 26) (status 800000))
+  (segment (start 46.99 57.785) (end 47.117 57.658) (width 0.25) (layer B.Cu) (net 26))
+  (segment (start 46.99 34.29) (end 46.99 57.785) (width 0.25) (layer B.Cu) (net 26))
+  (segment (start 57.15 24.13) (end 46.99 34.29) (width 0.25) (layer B.Cu) (net 26))
   (segment (start 59.69 24.13) (end 63.5 24.13) (width 0.25) (layer F.Cu) (net 26))
-  (segment (start 73.66 20.32) (end 88.9 20.32) (width 0.25) (layer F.Cu) (net 26))
-  (segment (start 88.9 43.18) (end 86.36 43.18) (width 0.25) (layer F.Cu) (net 26))
-  (segment (start 88.9 20.32) (end 88.9 43.18) (width 0.25) (layer F.Cu) (net 26))
-  (segment (start 73.66 20.32) (end 68.58 20.32) (width 0.25) (layer F.Cu) (net 26))
   (zone (net 26) (net_name +12V) (layer F.Cu) (hatch edge 0.508)
     (connect_pads (clearance 0.508))
