File: PCB/mainpcb.sch (KiCad schematic (older format))
At the start: 10 parts, among them CON1 BARREL_JACK, P1 VALVE1, P2 VALVE2, Q1 PN2222A, Q2 PN2222A, U1 LM317T, U2 Adafruit_HUZZAH

Commit message: structure changes
Parts:
- U2: footprint Adafruit_huzzah:Adafruit HUZZAH -> myparts:Adafruit-HUZZAH
Connections:
- net GND: now reaches CON1.2, Q1.1 (E), Q2.1 (E), R2.2, U2.19 (GND)
- net +12V: now reaches P1.1 (P1), P2.1 (P1), R11.1, U1.2 (OUT), U2.15 (VIN)
Changed lines of the file:
@@
 EESchema Schematic File Version 2
+LIBS:myparts
 LIBS:power
 LIBS:device
@@
 F 0 "U2" H 5500 2950 60  0000 C CNN
 F 1 "Adafruit_HUZZAH" H 5500 4150 60  0000 C CNN
-F 2 "Adafruit_huzzah:Adafruit HUZZAH" H 5400 3200 60  0001 C CNN
+F 2 "myparts:Adafruit-HUZZAH" H 5400 3200 60  0001 C CNN
 F 3 "" H 5400 3200 60  0000 C CNN
 	1    5500 3550
@@
 	3550 2500 4000 2500
 Wire Wire Line
-	2750 1950 2750 2800
+	2750 1950 2750 3000
 Wire Wire Line
 	2750 2800 6100 2800
@@
 Connection ~ 5100 1750
 Wire Wire Line
-	4900 3800 4300 3800
-Wire Wire Line
-	4300 3800 4300 1750
+	4300 3800 4900 3800
+Wire Wire Line
+	4300 1450 4300 3800
 Connection ~ 4300 1750
 Wire Wire Line
@@
 Wire Wire Line
 	4650 3400 4900 3400
+$Comp
+L GND #PWR01
+U 1 1 56FAB0DF
+P 2750 3000
+F 0 "#PWR01" H 2750 2750 50  0001 C CNN
+F 1 "GND" H 2750 2850 50  0000 C CNN
+F 2 "" H 2750 3000 50  0000 C CNN
+F 3 "" H 2750 3000 50  0000 C CNN
+	1    2750 3000
+	1    0    0    -1
+$EndComp
+Connection ~ 2750 2800
+$Comp
+L +12V #PWR02
+U 1 1 56FAB133
+P 4300 1450
+F 0 "#PWR02" H 4300 1300 50  0001 C CNN
+F 1 "+12V" H 4300 1590 50  0000 C CNN
+F 2 "" H 4300 1450 50  0000 C CNN
+F 3 "" H 4300 1450 50  0000 C CNN
+	1    4300 1450
+	1    0    0    -1
+$EndComp
 $EndSCHEMATC
